Commit message: Model loads in Gazebo; stuff "works"

File: chimera_description/urdf/chimera.urdf.xacro (robot description, xacro)
@@ -1,5 +1,25 @@
 <?xml version="1.0"?>
-<robot  xmlns:xacro="http://www.ros.org/wiki/xacro" name="chimera" >
+<robot xmlns:xacro="http://www.ros.org/wiki/xacro" name="chimera" >
   <xacro:property name="width" value=".2" />
+  <!-- Copied from https://github.com/elephantrobotics/mycobot_ros/pull/47/files#diff-376dbc4a3acb2831ff5adea9612541636ce126703a5f9477713e5dd388a4e196 -->
+  <xacro:macro name="box_inertial" params="mass x y z">
+    <inertial>
+      <mass value="${mass}" />
+      <inertia ixx="${mass*(y*y+z*z)/12}" ixy = "0" ixz = "0"
+      iyy="${mass*(z*z+x*x)/12}" iyz = "0"
+      izz="${mass*(x*x+y*y)/12}" />
+    </inertial>
+  </xacro:macro>
+  <xacro:macro name="cylinder_inertia" params="mass r h">
+    <inertia ixx="${mass*(3*r*r+h*h)/12}" ixy="0" ixz="0"
+      iyy="${mass*(3*r*r+h*h)/12}" iyz="0"
+      izz="${mass*r*r/2}" />
+  </xacro:macro>
+  <xacro:macro name="def_inertial" params="mass">
+    <inertial>
+      <mass value="${mass}" />
+      <inertia ixx="1.0" ixy="0.0" ixz="0.0" iyy="1.0" iyz="0.0" izz="1.0" />
+    </inertial>
+  </xacro:macro>
   <link name="base_footprint"/>
   <link name="base_link">
@@ -8,5 +28,5 @@
 	<mesh filename="package://chimera_description/meshes/base_link.stl"/>
       </geometry>
-      <origin xyz = "0.0 0 0 " rpy = "0 0 0"/>
+      <origin xyz = "0.0 0.0 0.0 " rpy = "0 0 0"/>
       <material name="">
 	<color rgba="0 0.7 0 1"/>
@@ -18,4 +38,5 @@
       </geometry>
     </collision>
+    <xacro:box_inertial mass="5.0" x="0.30" y="0.24" z="0.10"/>
   </link>
   <link name="joint1">
@@ -34,4 +55,5 @@
         <origin xyz = "0.0 0 0 " rpy = " 0 0 3.14159"/>
     </collision>
+    <xacro:def_inertial mass="0.5"/>
   </link>
   <link name="joint2">
@@ -48,4 +70,5 @@
       <origin xyz = "0.0 0 -0.06096 " rpy = " 0 0 -1.5708"/>
     </collision>
+    <xacro:def_inertial mass="0.3"/>
   </link>
   <link name="joint3">
@@ -62,9 +85,9 @@
       <origin xyz = "0.0 0 0.03256 " rpy = " 0 -1.5708 0"/>
     </collision>
+    <xacro:def_inertial mass="0.2"/>
   </link>
   <link name="joint4">
     <visual>
       <geometry>
-       <!--- 0.0 0 -0.04 -->
        <mesh filename="package://chimera_description/meshes/joint4.dae"/>
       </geometry>
@@ -73,14 +96,13 @@
     <collision>
       <geometry>
-       <!--- 0.0 0 -0.04 -->
        <mesh filename="package://chimera_description/meshes/joint4.dae"/>
       </geometry>
       <origin xyz = "0.0 0 0.03056 " rpy = " 0 -1.5708 0"/>
     </collision>
+    <xacro:def_inertial mass="0.2"/>
   </link>
   <link name="joint5">
     <visual>
       <geometry>
-       <!--- 0.0 0 -0.04 -->
        <mesh filename="package://chimera_description/meshes/joint5.dae"/>
       </geometry>
@@ -89,14 +111,13 @@
     <collision>
        <geometry>
-       <!--- 0.0 0 -0.04 -->
        <mesh filename="package://chimera_description/meshes/joint5.dae"/>
       </geometry>
       <origin xyz = "0.0 0 -0.03356 " rpy = " -1.5708 0 0"/>
     </collision>
+    <xacro:def_inertial mass="0.25"/>
   </link>
   <link name="joint6">
     <visual>
       <geometry>
-       <!--- 0.0 0 -0.04 -->
        <mesh filename="package://chimera_description/meshes/joint6.dae"/>
       </geometry>
@@ -105,14 +126,13 @@
     <collision>
       <geometry>
-       <!--- 0.0 0 -0.04 -->
        <mesh filename="package://chimera_description/meshes/joint6.dae"/>
       </geometry>
     <origin xyz = "0 0.00 -0.038 " rpy = " 0 0 0"/>
     </collision>
+    <xacro:def_inertial mass="0.1"/>
   </link>
   <link name="joint6_flange">
     <visual>
       <geometry>
-       <!--- 0.0 0 -0.04 -->
        <mesh filename="package://chimera_description/meshes/joint7.dae"/>
       </geometry>
@@ -121,9 +141,78 @@
     <collision>
       <geometry>
-       <!--- 0.0 0 -0.04 -->
        <mesh filename="package://chimera_description/meshes/joint7.dae"/>
       </geometry>
     <origin xyz = "0.0 0 -0.012 " rpy = " 0 0 0"/>
     </collision>
+    <xacro:def_inertial mass="0.05"/>
+  </link>
+  <link name="left_front_wheel">
+    <!--
+    <visual>
+      <origin rpy="1.57075 0 0" xyz="0 0 0"/>
+      <geometry>
+        <cylinder length="0.05" radius="0.05"/>
+      </geometry>
+      <material name="black"/>
+    </visual>
+    -->
+    <xacro:def_inertial mass="0.1"/>
+  </link>
+  <link name="left_mid_wheel">
+    <!--
+    <visual>
+      <origin rpy="1.57075 0 0" xyz="0 0 0"/>
+      <geometry>
+        <cylinder length="0.05" radius="0.05"/>
+      </geometry>
+      <material name="black"/>
+    </visual>
+    -->
+    <xacro:def_inertial mass="0.1"/>
+  </link>
+  <link name="left_back_wheel">
+    <!--
+    <visual>
+      <origin rpy="1.57075 0 0" xyz="0 0 0"/>
+      <geometry>
+        <cylinder length="0.05" radius="0.05"/>
+      </geometry>
+      <material name="black"/>
+    </visual>
+    -->
+    <xacro:def_inertial mass="0.1"/>
+  </link>
+  <link name="right_front_wheel">
+    <!--
+    <visual>
+      <origin rpy="1.57075 0 0" xyz="0 0 0"/>
+      <geometry>
+        <cylinder length="0.05" radius="0.05"/>
+      </geometry>
+      <material name="black"/>
+    </visual> -->
+    <xacro:def_inertial mass="0.1"/>
+  </link>
+  <link name="right_mid_wheel">
+    <!--
+    <visual>
+      <origin rpy="1.57075 0 0" xyz="0 0 0"/>
+      <geometry>
+        <cylinder length="0.05" radius="0.05"/>
+      </geometry>
+      <material name="black"/>
+    </visual> -->
+    <xacro:def_inertial mass="0.1"/>
+  </link>
+  <link name="right_back_wheel">
+    <!--
+    <visual>
+      <origin rpy="1.57075 0 0" xyz="0 0 0"/>
+      <geometry>
+        <cylinder length="0.05" radius="0.05"/>
+      </geometry>
+      <material name="black"/>
+    </visual> -->
+    <xacro:def_inertial mass="0.1"/>
   </link>
   <joint name="joint2_to_joint1" type="revolute">
@@ -147,95 +236,4 @@
     <child link="joint4"/>
     <origin xyz= "  -0.1104 0 0   " rpy = "0 0 0"/>
-  </joint>
-  <!-- wheels -->
-  <link name="left_front_wheel">
-    <visual>
-      <origin rpy="1.57075 0 0" xyz="0 0 0"/>
-      <geometry>
-        <cylinder length="0.05" radius="0.05"/>
-      </geometry>
-      <material name="black"/>
-    </visual>
-  </link>
-  <link name="left_mid_wheel">
-    <visual>
-      <origin rpy="1.57075 0 0" xyz="0 0 0"/>
-      <geometry>
-        <cylinder length="0.05" radius="0.05"/>
-      </geometry>
-      <material name="black"/>
-    </visual>
-  </link>
-  <link name="left_back_wheel">
-    <visual>
-      <origin rpy="1.57075 0 0" xyz="0 0 0"/>
-      <geometry>
-        <cylinder length="0.05" radius="0.05"/>
-      </geometry>
-      <material name="black"/>
-    </visual>
-  </link>
-  <joint name="left_front_wheel_joint" type="continuous">
-    <axis rpy="0 0 0" xyz="0 1 0"/>
-    <parent link="base_link"/>
-    <child link="left_front_wheel"/>
-    <origin rpy="0 0 0" xyz="0.12 0.09 -0.03"/>
-  </joint>
-  <joint name="left_mid_wheel_joint" type="continuous">
-    <axis rpy="0 0 0" xyz="0 1 0"/>
-    <parent link="base_link"/>
-    <child link="left_mid_wheel"/>
-    <origin rpy="0 0 0" xyz="0.0 0.09 -0.03"/>
-  </joint>
-  <joint name="left_back_wheel_joint" type="continuous">
-    <axis rpy="0 0 0" xyz="0 1 0"/>
-    <parent link="base_link"/>
-    <child link="left_back_wheel"/>
-    <origin rpy="0 0 0" xyz="-0.12 0.09 -0.03"/>
-  </joint>
-  <link name="right_front_wheel">
-    <visual>
-      <origin rpy="1.57075 0 0" xyz="0 0 0"/>
-      <geometry>
-        <cylinder length="0.05" radius="0.05"/>
-      </geometry>
-      <material name="black"/>
-    </visual>
-  </link>
-  <link name="right_mid_wheel">
-    <visual>
-      <origin rpy="1.57075 0 0" xyz="0 0 0"/>
-      <geometry>
-        <cylinder length="0.05" radius="0.05"/>
-      </geometry>
-      <material name="black"/>
-    </visual>
-  </link>
-  <link name="right_back_wheel">
-    <visual>
-      <origin rpy="1.57075 0 0" xyz="0 0 0"/>
-      <geometry>
-        <cylinder length="0.05" radius="0.05"/>
-      </geometry>
-      <material name="black"/>
-    </visual>
-  </link>
-  <joint name="right_front_wheel_joint" type="continuous">
-    <axis rpy="0 0 0" xyz="0 1 0"/>
-    <parent link="base_link"/>
-    <child link="right_front_wheel"/>
-    <origin rpy="0 0 0" xyz="0.12 -0.09 -0.03"/>
-  </joint>
-  <joint name="right_mid_wheel_joint" type="continuous">
-    <axis rpy="0 0 0" xyz="0 1 0"/>
-    <parent link="base_link"/>
-    <child link="right_mid_wheel"/>
-    <origin rpy="0 0 0" xyz="0.0 -0.09 -0.03"/>
-  </joint>
-  <joint name="right_back_wheel_joint" type="continuous">
-    <axis rpy="0 0 0" xyz="0 1 0"/>
-    <parent link="base_link"/>
-    <child link="right_back_wheel"/>
-    <origin rpy="0 0 0" xyz="-0.12 -0.09 -0.03"/>
   </joint>
   <joint name="joint5_to_joint4" type="revolute">
@@ -270,3 +268,39 @@
     <origin xyz="-0.03 0.0 0.087" rpy="0 0 0"/>
   </joint>
+  <joint name="left_front_wheel_joint" type="continuous">
+    <axis rpy="0 0 0" xyz="0 1 0"/>
+    <parent link="base_link"/>
+    <child link="left_front_wheel"/>
+    <origin rpy="0 0 0" xyz="0.12 0.09 -0.03"/>
+  </joint>
+  <joint name="left_mid_wheel_joint" type="continuous">
+    <axis rpy="0 0 0" xyz="0 1 0"/>
+    <parent link="base_link"/>
+    <child link="left_mid_wheel"/>
+    <origin rpy="0 0 0" xyz="0.0 0.09 -0.03"/>
+  </joint>
+  <joint name="left_back_wheel_joint" type="continuous">
+    <axis rpy="0 0 0" xyz="0 1 0"/>
+    <parent link="base_link"/>
+    <child link="left_back_wheel"/>
+    <origin rpy="0 0 0" xyz="-0.12 0.09 -0.03"/>
+  </joint>
+  <joint name="right_front_wheel_joint" type="continuous">
+    <axis rpy="0 0 0" xyz="0 1 0"/>
+    <parent link="base_link"/>
+    <child link="right_front_wheel"/>
+    <origin rpy="0 0 0" xyz="0.12 -0.09 -0.03"/>
+  </joint>
+  <joint name="right_mid_wheel_joint" type="continuous">
+    <axis rpy="0 0 0" xyz="0 1 0"/>
+    <parent link="base_link"/>
+    <child link="right_mid_wheel"/>
+    <origin rpy="0 0 0" xyz="0.0 -0.09 -0.03"/>
+  </joint>
+  <joint name="right_back_wheel_joint" type="continuous">
+    <axis rpy="0 0 0" xyz="0 1 0"/>
+    <parent link="base_link"/>
+    <child link="right_back_wheel"/>
+    <origin rpy="0 0 0" xyz="-0.12 -0.09 -0.03"/>
+  </joint>
 </robot>

Commit message: Inertial parameters and accurate weights

File: chimera_description/urdf/chimera.urdf.xacro (robot description, xacro)
@@ -2,24 +2,22 @@
 <robot xmlns:xacro="http://www.ros.org/wiki/xacro" name="chimera" >
   <xacro:property name="width" value=".2" />
-  <!-- Copied from https://github.com/elephantrobotics/mycobot_ros/pull/47/files#diff-376dbc4a3acb2831ff5adea9612541636ce126703a5f9477713e5dd388a4e196 -->
-  <xacro:macro name="box_inertial" params="mass x y z">
+  <!-- Copied from https://github.com/elephantrobotics/mycobot_ros/pull/47/files#diff-376dbc4a3acb2831ff5adea9612541636ce126703a5f9477713e5dd388a4e196. Can be found here: https://en.wikipedia.org/wiki/List_of_moments_of_inertia#List_of_3D_inertia_tensors as well.-->
+  <xacro:macro name="box_inertial" params="m w d h">
     <inertial>
-      <mass value="${mass}" />
-      <inertia ixx="${mass*(y*y+z*z)/12}" ixy = "0" ixz = "0"
-      iyy="${mass*(z*z+x*x)/12}" iyz = "0"
-      izz="${mass*(x*x+y*y)/12}" />
+      <mass value="${m}" />
+      <inertia ixx="${m*(h*h + d*d)/12}" ixy = "0" ixz = "0"
+      iyy="${m*(h*h+w*w)/12}" iyz = "0"
+      izz="${m*(w*w+d*d)/12}" />
     </inertial>
   </xacro:macro>
-  <xacro:macro name="cylinder_inertia" params="mass r h">
-    <inertia ixx="${mass*(3*r*r+h*h)/12}" ixy="0" ixz="0"
-      iyy="${mass*(3*r*r+h*h)/12}" iyz="0"
-      izz="${mass*r*r/2}" />
-  </xacro:macro>
-  <xacro:macro name="def_inertial" params="mass">
+  <xacro:macro name="hcylinder_inertial" params="m r h">
     <inertial>
-      <mass value="${mass}" />
-      <inertia ixx="1.0" ixy="0.0" ixz="0.0" iyy="1.0" iyz="0.0" izz="1.0" />
+      <mass value="${m}" />
+      <inertia ixx="${m*(3*(r*r)+h*h)/12}" ixy = "0" ixz = "0"
+      iyy="${m*(3*(r*r)+h*h)/12}" iyz = "0"
+      izz="${m*(r*r)/12}" />
     </inertial>
   </xacro:macro>
+  <!-- The joints are modelled as a cylinder, that encompasses the whole joint. -->
   <link name="base_footprint"/>
   <link name="base_link">
@@ -38,10 +36,9 @@
       </geometry>
     </collision>
-    <xacro:box_inertial mass="5.0" x="0.30" y="0.24" z="0.10"/>
+    <xacro:box_inertial m="5.5" w="0.24" d="0.3" h="0.10"/>
   </link>
   <link name="joint1">
     <visual>
       <geometry>
-	     <!--- 0.0 0 -0.04  1.5708 3.14159-->
        <mesh filename="package://chimera_description/meshes/joint1.dae"/>
       </geometry>
@@ -50,10 +47,9 @@
     <collision>
       <geometry>
-	     <!--- 0.0 0 -0.04  1.5708 3.14159-->
        <mesh filename="package://chimera_description/meshes/joint1.dae"/>
         </geometry>
         <origin xyz = "0.0 0 0 " rpy = " 0 0 3.14159"/>
     </collision>
-    <xacro:def_inertial mass="0.5"/>
+    <xacro:hcylinder_inertial m="1.0" r="0.045" h="0.073"/>
   </link>
   <link name="joint2">
@@ -70,6 +66,7 @@
       <origin xyz = "0.0 0 -0.06096 " rpy = " 0 0 -1.5708"/>
     </collision>
-    <xacro:def_inertial mass="0.3"/>
-  </link>
+    <xacro:hcylinder_inertial m="0.1" r="0.025" h="0.087"/>
+  </link>
+  <!--
   <link name="joint3">
     <visual>
@@ -85,5 +82,5 @@
       <origin xyz = "0.0 0 0.03256 " rpy = " 0 -1.5708 0"/>
     </collision>
-    <xacro:def_inertial mass="0.2"/>
+    <xacro:hcylinder_inertial m="0.2" r="0.03" h="0.155"/>
   </link>
   <link name="joint4">
@@ -100,5 +97,5 @@
       <origin xyz = "0.0 0 0.03056 " rpy = " 0 -1.5708 0"/>
     </collision>
-    <xacro:def_inertial mass="0.2"/>
+    <xacro:hcylinder_inertial m="0.18" r="0.0275" h="0.136"/>
   </link>
   <link name="joint5">
@@ -115,5 +112,5 @@
       <origin xyz = "0.0 0 -0.03356 " rpy = " -1.5708 0 0"/>
     </collision>
-    <xacro:def_inertial mass="0.25"/>
+    <xacro:hcylinder_inertial m="0.1" r="0.0275" h="0.06"/>
   </link>
   <link name="joint6">
@@ -130,5 +127,5 @@
     <origin xyz = "0 0.00 -0.038 " rpy = " 0 0 0"/>
     </collision>
-    <xacro:def_inertial mass="0.1"/>
+    <xacro:hcylinder_inertial m="0.1" r="0.018" h="0.06"/>
   </link>
   <link name="joint6_flange">
@@ -145,117 +142,7 @@
     <origin xyz = "0.0 0 -0.012 " rpy = " 0 0 0"/>
     </collision>
-    <xacro:def_inertial mass="0.05"/>
-  </link>
-  <link name="left_front_wheel">
-    <!--
-    <visual>
-      <origin rpy="1.57075 0 0" xyz="0 0 0"/>
-      <geometry>
-        <cylinder length="0.05" radius="0.05"/>
-      </geometry>
-      <material name="black"/>
-    </visual>
-    -->
-    <xacro:def_inertial mass="0.1"/>
-  </link>
-  <link name="left_mid_wheel">
-    <!--
-    <visual>
-      <origin rpy="1.57075 0 0" xyz="0 0 0"/>
-      <geometry>
-        <cylinder length="0.05" radius="0.05"/>
-      </geometry>
-      <material name="black"/>
-    </visual>
-    -->
-    <xacro:def_inertial mass="0.1"/>
-  </link>
-  <link name="left_back_wheel">
-    <!--
-    <visual>
-      <origin rpy="1.57075 0 0" xyz="0 0 0"/>
-      <geometry>
-        <cylinder length="0.05" radius="0.05"/>
-      </geometry>
-      <material name="black"/>
-    </visual>
-    -->
-    <xacro:def_inertial mass="0.1"/>
-  </link>
-  <link name="right_front_wheel">
-    <!--
-    <visual>
-      <origin rpy="1.57075 0 0" xyz="0 0 0"/>
-      <geometry>
-        <cylinder length="0.05" radius="0.05"/>
-      </geometry>
-      <material name="black"/>
-    </visual> -->
-    <xacro:def_inertial mass="0.1"/>
-  </link>
-  <link name="right_mid_wheel">
-    <!--
-    <visual>
-      <origin rpy="1.57075 0 0" xyz="0 0 0"/>
-      <geometry>
-        <cylinder length="0.05" radius="0.05"/>
-      </geometry>
-      <material name="black"/>
-    </visual> -->
-    <xacro:def_inertial mass="0.1"/>
-  </link>
-  <link name="right_back_wheel">
-    <!--
-    <visual>
-      <origin rpy="1.57075 0 0" xyz="0 0 0"/>
-      <geometry>
-        <cylinder length="0.05" radius="0.05"/>
-      </geometry>
-      <material name="black"/>
-    </visual> -->
-    <xacro:def_inertial mass="0.1"/>
-  </link>
-  <joint name="joint2_to_joint1" type="revolute">
-    <axis xyz="0 0 1"/>
-    <limit effort = "1000.0" lower = "-3.14" upper = "3.14159" velocity = "0"/>
-    <parent link="joint1"/>
-    <child link="joint2"/>
-    <origin xyz= "0 0 0.13156" rpy = "0 0 1.5708"/>
-  </joint>
-  <joint name="joint3_to_joint2" type="revolute">
-    <axis xyz="0 0 1"/>
-    <limit effort = "1000.0" lower = "-3.14" upper = "3.14159" velocity = "0"/>
-    <parent link="joint2"/>
-    <child link="joint3"/>
-    <origin xyz= "0 0  0" rpy = "0 1.5708 -1.5708"/>
-  </joint>
-  <joint name="joint4_to_joint3" type="revolute">
-    <axis xyz=" 0 0 1"/>
-    <limit effort = "1000.0" lower = "-3.14" upper = "3.14159" velocity = "0"/>
-    <parent link="joint3"/>
-    <child link="joint4"/>
-    <origin xyz= "  -0.1104 0 0   " rpy = "0 0 0"/>
-  </joint>
-  <joint name="joint5_to_joint4" type="revolute">
-    <axis xyz=" 0 0 1"/>
-    <limit effort = "1000.0" lower = "-3.14" upper = "3.14159" velocity = "0"/>
-    <parent link="joint4"/>
-    <child link="joint5"/>
-    <origin xyz= "-0.096 0 0.06462" rpy = "0 0 -1.5708"/>
-  </joint>
-  <joint name="joint6_to_joint5" type="revolute">
-    <axis xyz="0 0 1"/>
-    <limit effort = "1000.0" lower = "-3.14" upper = "3.14159" velocity = "0"/>
-    <parent link="joint5"/>
-    <child link="joint6"/>
-    <origin xyz= "0 -0.07318 0" rpy = "1.5708 -1.5708 0"/>
-  </joint>
-  <joint name="joint6output_to_joint6" type="revolute">
-    <axis xyz="0 0 1"/>
-    <limit effort = "1000.0" lower = "-3.14" upper = "3.14159" velocity = "0"/>
-    <parent link="joint6"/>
-    <child link="joint6_flange"/>
-    <origin xyz= "0 0.0456 0" rpy = "-1.5708 0 0"/>
-  </joint>
+    <xacro:hcylinder_inertial m="0.05" r="0.018" h="0.02"/>
+  </link>
+-->
   <joint name="base_joint" type="fixed">
     <parent link="base_footprint"/>
@@ -268,39 +155,47 @@
     <origin xyz="-0.03 0.0 0.087" rpy="0 0 0"/>
   </joint>
-  <joint name="left_front_wheel_joint" type="continuous">
-    <axis rpy="0 0 0" xyz="0 1 0"/>
-    <parent link="base_link"/>
-    <child link="left_front_wheel"/>
-    <origin rpy="0 0 0" xyz="0.12 0.09 -0.03"/>
-  </joint>
-  <joint name="left_mid_wheel_joint" type="continuous">
-    <axis rpy="0 0 0" xyz="0 1 0"/>
-    <parent link="base_link"/>
-    <child link="left_mid_wheel"/>
-    <origin rpy="0 0 0" xyz="0.0 0.09 -0.03"/>
-  </joint>
-  <joint name="left_back_wheel_joint" type="continuous">
-    <axis rpy="0 0 0" xyz="0 1 0"/>
-    <parent link="base_link"/>
-    <child link="left_back_wheel"/>
-    <origin rpy="0 0 0" xyz="-0.12 0.09 -0.03"/>
-  </joint>
-  <joint name="right_front_wheel_joint" type="continuous">
-    <axis rpy="0 0 0" xyz="0 1 0"/>
-    <parent link="base_link"/>
-    <child link="right_front_wheel"/>
-    <origin rpy="0 0 0" xyz="0.12 -0.09 -0.03"/>
-  </joint>
-  <joint name="right_mid_wheel_joint" type="continuous">
-    <axis rpy="0 0 0" xyz="0 1 0"/>
-    <parent link="base_link"/>
-    <child link="right_mid_wheel"/>
-    <origin rpy="0 0 0" xyz="0.0 -0.09 -0.03"/>
-  </joint>
-  <joint name="right_back_wheel_joint" type="continuous">
-    <axis rpy="0 0 0" xyz="0 1 0"/>
-    <parent link="base_link"/>
-    <child link="right_back_wheel"/>
-    <origin rpy="0 0 0" xyz="-0.12 -0.09 -0.03"/>
-  </joint>
+  <joint name="joint2_to_joint1" type="revolute">
+    <axis xyz="0 0 1"/>
+    <limit effort = "1000.0" lower = "-3.14" upper = "3.14159" velocity = "0"/>
+    <parent link="joint1"/>
+    <child link="joint2"/>
+    <origin xyz= "0 0 0.13156" rpy = "0 0 1.5708"/>
+  </joint>
+<!--
+  <joint name="joint3_to_joint2" type="revolute">
+    <axis xyz="0 0 1"/>
+    <limit effort = "1000.0" lower = "-3.14" upper = "3.14159" velocity = "0"/>
+    <parent link="joint2"/>
+    <child link="joint3"/>
+    <origin xyz= "0 0  0" rpy = "0 1.5708 -1.5708"/>
+  </joint>
+  <joint name="joint4_to_joint3" type="revolute">
+    <axis xyz=" 0 0 1"/>
+    <limit effort = "1000.0" lower = "-3.14" upper = "3.14159" velocity = "0"/>
+    <parent link="joint3"/>
+    <child link="joint4"/>
+    <origin xyz= "  -0.1104 0 0   " rpy = "0 0 0"/>
+  </joint>
+  <joint name="joint5_to_joint4" type="revolute">
+    <axis xyz=" 0 0 1"/>
+    <limit effort = "1000.0" lower = "-3.14" upper = "3.14159" velocity = "0"/>
+    <parent link="joint4"/>
+    <child link="joint5"/>
+    <origin xyz= "-0.096 0 0.06462" rpy = "0 0 -1.5708"/>
+  </joint>
+  <joint name="joint6_to_joint5" type="revolute">
+    <axis xyz="0 0 1"/>
+    <limit effort = "1000.0" lower = "-3.14" upper = "3.14159" velocity = "0"/>
+    <parent link="joint5"/>
+    <child link="joint6"/>
+    <origin xyz= "0 -0.07318 0" rpy = "1.5708 -1.5708 0"/>
+  </joint>
+  <joint name="joint6output_to_joint6" type="revolute">
+    <axis xyz="0 0 1"/>
+    <limit effort = "1000.0" lower = "-3.14" upper = "3.14159" velocity = "0"/>
+    <parent link="joint6"/>
+    <child link="joint6_flange"/>
+    <origin xyz= "0 0.0456 0" rpy = "-1.5708 0 0"/>
+  </joint>
+-->
 </robot>
