Commit message: Updated meshes and URDF for tracks

File: chimera_description/urdf/chimera.urdf.xacro (robot description, xacro)
@@ -19,5 +19,13 @@
     </inertial>
   </xacro:macro>
-  <!-- The joints are modelled as a cylinder, that encompasses the whole joint. -->
+  <xacro:macro name="track_inertial">
+    <inertial>
+      <mass value="0.8" />
+      <inertia
+          ixx="0.01" ixy="0.0" ixz="0.0"
+          iyy="0.07" iyz="0.0"
+          izz="0.07"/>
+    </inertial>
+  </xacro:macro>
   <link name="base_footprint"/>
   <link name="base_link">
@@ -36,5 +44,5 @@
       </geometry>
     </collision>
-    <xacro:box_inertial m="5.5" w="0.24" d="0.34" h="0.15"/>
+    <xacro:box_inertial m="4.0" w="0.24" d="0.34" h="0.15"/>
   </link>
   <link name="joint1">
@@ -53,4 +61,5 @@
     <xacro:box_inertial m="0.25" w="0.1" d="0.1" h="0.1"/>
   </link>
+  <!-- TODO: Adding all the other joints -->
   <link name="joint2">
     <visual>
@@ -68,4 +77,5 @@
     <xacro:hcylinder_inertial m="0.1" r="0.025" h="0.087"/>
   </link>
+<!--
   <link name="joint3">
     <visual>
@@ -143,4 +153,75 @@
     <xacro:hcylinder_inertial m="0.05" r="0.018" h="0.02"/>
   </link>
+  -->
+  <link name="left_track">
+    <visual>
+      <geometry>
+       <mesh filename="package://chimera_description/meshes/track.stl"/>
+      </geometry>
+      <origin xyz="0.125 0.042 -0.01" rpy="0 0 0"/>
+      <material name="grey"/>
+    </visual>
+    <collision>
+      <geometry>
+       <mesh filename="package://chimera_description/meshes/track.stl"/>
+      </geometry>
+      <origin xyz="0.125 0.042 -0.01" rpy="0 0 0"/>
+    </collision>
+    <surface>
+      <friction>
+        <ode>
+          <mu>0.65</mu>
+          <mu2>0.85</mu2>
+        </ode>
+      </friction>
+      <contact>
+        <ode/>
+      </contact>
+    </surface>
+    <max_contacts>20</max_contacts>
+    <xacro:track_inertial />
+  </link>
+  <link name="right_track">
+    <visual>
+      <geometry>
+       <mesh filename="package://chimera_description/meshes/track.stl"/>
+      </geometry>
+      <origin xyz="0.125 -0.042 -0.01" rpy="0 0 0"/>
+      <material name="grey"/>
+    </visual>
+    <collision>
+      <geometry>
+       <mesh filename="package://chimera_description/meshes/track.stl"/>
+      </geometry>
+      <origin xyz="0.125 -0.042 -0.01" rpy="0 0 0"/>
+    </collision>
+    <surface>
+      <friction>
+        <ode>
+          <mu>0.65</mu>
+          <mu2>0.85</mu2>
+        </ode>
+      </friction>
+      <contact>
+        <ode/>
+      </contact>
+    </surface>
+    <max_contacts>20</max_contacts>
+    <xacro:track_inertial />
+  </link>
+  <joint name="right_track_motor" type="revolute">
+    <parent link="base_link"/>
+    <child link="right_track"/>
+    <axis xyz="0 1 0"/>
+    <origin xyz="-0.125 -0.05 -0.022" rpy="0 0 0"/>
+    <limit effort="100" velocity="10.0" lower="0" upper="0"/>
+  </joint>
+  <joint name="left_track_motor" type="revolute">
+    <parent link="base_link"/>
+    <child link="left_track"/>
+    <axis xyz="0 1 0"/>
+    <origin xyz="-0.125 0.05 -0.022" rpy="0 0 0"/>
+    <limit effort="100" velocity="10.0" lower="0" upper="0"/>
+  </joint>
   <joint name="base_joint" type="fixed">
     <parent link="base_footprint"/>
@@ -148,5 +229,5 @@
     <origin xyz="0.0 0.0 0.08" rpy="0 0 0"/>
   </joint>
-  <joint name="base_link_to_arm" type="fixed">
+  <joint name="arm_to_baselink" type="fixed">
     <parent link="base_link"/>
     <child link="joint1"/>
@@ -160,4 +241,5 @@
     <origin xyz= "0 0 0.13156" rpy = "0 0 1.5708"/>
   </joint>
+  <!--
   <joint name="joint3_to_joint2" type="revolute">
     <axis xyz="0 0 1"/>
@@ -195,3 +277,4 @@
     <origin xyz= "0 0.0456 0" rpy = "-1.5708 0 0"/>
   </joint>
+  -->
 </robot>

Commit message: Tracks, work!

File: chimera_description/urdf/chimera.urdf.xacro (robot description, xacro)
@@ -28,4 +28,5 @@
     </inertial>
   </xacro:macro>
+  <!-- Heavily referenced from https://github.com/clubcapra/markhor -->
   <link name="base_footprint"/>
   <link name="base_link">
@@ -225,7 +226,7 @@
   </joint>
   <joint name="base_joint" type="fixed">
-    <parent link="base_footprint"/>
-    <child link="base_link"/>
-    <origin xyz="0.0 0.0 0.08" rpy="0 0 0"/>
+    <parent link="base_link"/>
+    <child link="base_footprint"/>
+    <origin xyz="0.0 0.0 -0.0678" rpy="0 0 0"/>
   </joint>
   <joint name="arm_to_baselink" type="fixed">
@@ -278,3 +279,42 @@
   </joint>
   -->
+  <transmission name="left_track_trans" type="SimpleTransmission">
+    <type>transmission_interface/SimpleTransmission</type>
+    <joint name="left_track_motor">
+      <hardwareInterface>hardware_interface/EffortJointInterface</hardwareInterface>
+    </joint>
+    <actuator name="left_track_motor_drive">
+      <mechanicalReduction>1</mechanicalReduction>
+    </actuator>
+  </transmission>
+  <transmission name="right_track_trans" type="SimpleTransmission">
+    <type>transmission_interface/SimpleTransmission</type>
+    <joint name="right_track_motor">
+      <hardwareInterface>hardware_interface/EffortJointInterface</hardwareInterface>
+    </joint>
+    <actuator name="right_track_motor_drive">
+      <mechanicalReduction>1</mechanicalReduction>
+    </actuator>
+  </transmission>
+  <gazebo>
+    <plugin name="gazebo_ros_control" filename="libgazebo_ros_control.so">
+      <robotNamespace></robotNamespace>
+    </plugin>
+    <plugin filename="libSimpleTrackedVehiclePlugin.so" name="simple_tracked_vehicle">
+      <body>base_link</body>
+      <left_track>left_track</left_track>
+      <right_track>right_track</right_track>
+      <track_mu>0.65</track_mu>
+      <track_mu2>0.85</track_mu2>
+      <tracks_separation>0.14</tracks_separation>
+      <robot_namespace>chimera</robot_namespace>
+    </plugin>
+    <plugin name='tracked_vehicle_interface' filename='libgazebo_ros_tracked_vehicle_interface.so'>
+      <commandROSTopic>/chimera/cmd_vel</commandROSTopic>
+      <commandIGNTopic>~/chimera/cmd_vel_twist</commandIGNTopic>
+      <robotBaseFrame>base_link</robotBaseFrame>
+      <tracks_separation>0.14</tracks_separation>
+      <publishOdomTF>false</publishOdomTF>
+    </plugin>
+  </gazebo>
 </robot>

Commit message: Xacrofied stuff

File: chimera_description/urdf/chimera.urdf.xacro (robot description, xacro)
@@ -2,31 +2,7 @@
 <robot xmlns:xacro="http://www.ros.org/wiki/xacro" name="chimera" >
   <xacro:property name="width" value=".2" />
-  <!-- Copied from https://github.com/elephantrobotics/mycobot_ros/pull/47/files#diff-376dbc4a3acb2831ff5adea9612541636ce126703a5f9477713e5dd388a4e196. Can be found here: https://en.wikipedia.org/wiki/List_of_moments_of_inertia#List_of_3D_inertia_tensors as well.-->
-  <xacro:macro name="box_inertial" params="m w d h">
-    <inertial>
-      <mass value="${m}" />
-      <inertia ixx="${m*(h*h + d*d)/12}" ixy = "0" ixz = "0"
-      iyy="${m*(h*h+w*w)/12}" iyz = "0"
-      izz="${m*(w*w+d*d)/12}" />
-    </inertial>
-  </xacro:macro>
-  <xacro:macro name="hcylinder_inertial" params="m r h">
-    <inertial>
-      <mass value="${m}" />
-      <inertia ixx="${m*(3*(r*r)+h*h)/12}" ixy = "0" ixz = "0"
-      iyy="${m*(3*(r*r)+h*h)/12}" iyz = "0"
-      izz="${m*(r*r)/12}" />
-    </inertial>
-  </xacro:macro>
-  <xacro:macro name="track_inertial">
-    <inertial>
-      <mass value="0.8" />
-      <inertia
-          ixx="0.01" ixy="0.0" ixz="0.0"
-          iyy="0.07" iyz="0.0"
-          izz="0.07"/>
-    </inertial>
-  </xacro:macro>
-  <!-- Heavily referenced from https://github.com/clubcapra/markhor -->
+  <xacro:include filename="$(find chimera_description)/urdf/inertial.xacro"/>
+  <xacro:include filename="$(find chimera_description)/urdf/mycobot280_arduino.urdf.xacro"/>
+  <xacro:include filename="$(find chimera_description)/urdf/tracks.urdf.xacro"/>
   <link name="base_footprint"/>
   <link name="base_link">
@@ -47,182 +23,7 @@
     <xacro:box_inertial m="4.0" w="0.24" d="0.34" h="0.15"/>
   </link>
-  <link name="joint1">
-    <visual>
-      <geometry>
-       <mesh filename="package://chimera_description/meshes/joint1.dae"/>
-      </geometry>
-      <origin xyz = "0.0 0 0 " rpy = " 0 0 3.14159"/>
-    </visual>
-    <collision>
-      <geometry>
-       <mesh filename="package://chimera_description/meshes/joint1.dae"/>
-        </geometry>
-        <origin xyz = "0.0 0 0 " rpy = " 0 0 3.14159"/>
-    </collision>
-    <xacro:box_inertial m="0.25" w="0.1" d="0.1" h="0.1"/>
-  </link>
-  <!-- TODO: Adding all the other joints -->
-  <link name="joint2">
-    <visual>
-      <geometry>
-       <mesh filename="package://chimera_description/meshes/joint2.dae"/>
-      </geometry>
-      <origin xyz = "0.0 0 -0.06096 " rpy = " 0 0 -1.5708"/>
-    </visual>
-    <collision>
-     <geometry>
-       <mesh filename="package://chimera_description/meshes/joint2.dae"/>
-      </geometry>
-      <origin xyz = "0.0 0 -0.06096 " rpy = " 0 0 -1.5708"/>
-    </collision>
-    <xacro:hcylinder_inertial m="0.1" r="0.025" h="0.087"/>
-  </link>
-<!--
-  <link name="joint3">
-    <visual>
-      <geometry>
-       <mesh filename="package://chimera_description/meshes/joint3.dae"/>
-      </geometry>
-    <origin xyz = "0.0 0 0.03256 " rpy = " 0 -1.5708 0"/>
-    </visual>
-    <collision>
-      <geometry>
-       <mesh filename="package://chimera_description/meshes/joint3.dae"/>
-      </geometry>
-      <origin xyz = "0.0 0 0.03256 " rpy = " 0 -1.5708 0"/>
-    </collision>
-    <xacro:hcylinder_inertial m="0.2" r="0.03" h="0.155"/>
-  </link>
-  <link name="joint4">
-    <visual>
-      <geometry>
-       <mesh filename="package://chimera_description/meshes/joint4.dae"/>
-      </geometry>
-      <origin xyz = "0.0 0 0.03056 " rpy = " 0 -1.5708 0"/>
-    </visual>
-    <collision>
-      <geometry>
-       <mesh filename="package://chimera_description/meshes/joint4.dae"/>
-      </geometry>
-      <origin xyz = "0.0 0 0.03056 " rpy = " 0 -1.5708 0"/>
-    </collision>
-    <xacro:hcylinder_inertial m="0.18" r="0.0275" h="0.136"/>
-  </link>
-  <link name="joint5">
-    <visual>
-      <geometry>
-       <mesh filename="package://chimera_description/meshes/joint5.dae"/>
-      </geometry>
-    <origin xyz = "0.0 0 -0.03356 " rpy = " -1.5708 0 0"/>
-    </visual>
-    <collision>
-       <geometry>
-       <mesh filename="package://chimera_description/meshes/joint5.dae"/>
-      </geometry>
-      <origin xyz = "0.0 0 -0.03356 " rpy = " -1.5708 0 0"/>
-    </collision>
-    <xacro:hcylinder_inertial m="0.1" r="0.0275" h="0.06"/>
-  </link>
-  <link name="joint6">
-    <visual>
-      <geometry>
-       <mesh filename="package://chimera_description/meshes/joint6.dae"/>
-      </geometry>
-    <origin xyz = "0 0.00 -0.038 " rpy = " 0 0 0"/>
-    </visual>
-    <collision>
-      <geometry>
-       <mesh filename="package://chimera_description/meshes/joint6.dae"/>
-      </geometry>
-    <origin xyz = "0 0.00 -0.038 " rpy = " 0 0 0"/>
-    </collision>
-    <xacro:hcylinder_inertial m="0.1" r="0.018" h="0.06"/>
-  </link>
-  <link name="joint6_flange">
-    <visual>
-      <geometry>
-       <mesh filename="package://chimera_description/meshes/joint7.dae"/>
-      </geometry>
-    <origin xyz = "0.0 0 -0.012 " rpy = " 0 0 0"/>
-    </visual>
-    <collision>
-      <geometry>
-       <mesh filename="package://chimera_description/meshes/joint7.dae"/>
-      </geometry>
-    <origin xyz = "0.0 0 -0.012 " rpy = " 0 0 0"/>
-    </collision>
-    <xacro:hcylinder_inertial m="0.05" r="0.018" h="0.02"/>
-  </link>
-  -->
-  <link name="left_track">
-    <visual>
-      <geometry>
-       <mesh filename="package://chimera_description/meshes/track.stl"/>
-      </geometry>
-      <origin xyz="0.125 0.042 -0.01" rpy="0 0 0"/>
-      <material name="grey"/>
-    </visual>
-    <collision>
-      <geometry>
-       <mesh filename="package://chimera_description/meshes/track.stl"/>
-      </geometry>
-      <origin xyz="0.125 0.042 -0.01" rpy="0 0 0"/>
-    </collision>
-    <surface>
-      <friction>
-        <ode>
-          <mu>0.65</mu>
-          <mu2>0.85</mu2>
-        </ode>
-      </friction>
-      <contact>
-        <ode/>
-      </contact>
-    </surface>
-    <max_contacts>20</max_contacts>
-    <xacro:track_inertial />
-  </link>
-  <link name="right_track">
-    <visual>
-      <geometry>
-       <mesh filename="package://chimera_description/meshes/track.stl"/>
-      </geometry>
-      <origin xyz="0.125 -0.042 -0.01" rpy="0 0 0"/>
-      <material name="grey"/>
-    </visual>
-    <collision>
-      <geometry>
-       <mesh filename="package://chimera_description/meshes/track.stl"/>
-      </geometry>
-      <origin xyz="0.125 -0.042 -0.01" rpy="0 0 0"/>
-    </collision>
-    <surface>
-      <friction>
-        <ode>
-          <mu>0.65</mu>
-          <mu2>0.85</mu2>
-        </ode>
-      </friction>
-      <contact>
-        <ode/>
-      </contact>
-    </surface>
-    <max_contacts>20</max_contacts>
-    <xacro:track_inertial />
-  </link>
-  <joint name="right_track_motor" type="revolute">
-    <parent link="base_link"/>
-    <child link="right_track"/>
-    <axis xyz="0 1 0"/>
-    <origin xyz="-0.125 -0.05 -0.022" rpy="0 0 0"/>
-    <limit effort="100" velocity="10.0" lower="0" upper="0"/>
-  </joint>
-  <joint name="left_track_motor" type="revolute">
-    <parent link="base_link"/>
-    <child link="left_track"/>
-    <axis xyz="0 1 0"/>
-    <origin xyz="-0.125 0.05 -0.022" rpy="0 0 0"/>
-    <limit effort="100" velocity="10.0" lower="0" upper="0"/>
-  </joint>
+  <xacro:my_cobot_arm moving_base_link="base_link"
+		      originxyz="-0.03 0.0 0.087" originrpy="0 0 0"/>
+  <xacro:tracks />
   <joint name="base_joint" type="fixed">
     <parent link="base_link"/>
@@ -230,90 +31,7 @@
     <origin xyz="0.0 0.0 -0.0678" rpy="0 0 0"/>
   </joint>
-  <joint name="arm_to_baselink" type="fixed">
-    <parent link="base_link"/>
-    <child link="joint1"/>
-    <origin xyz="-0.03 0.0 0.087" rpy="0 0 0"/>
-  </joint>
-  <joint name="joint2_to_joint1" type="revolute">
-    <axis xyz="0 0 1"/>
-    <limit effort = "1000.0" lower = "-3.14" upper = "3.14159" velocity = "0"/>
-    <parent link="joint1"/>
-    <child link="joint2"/>
-    <origin xyz= "0 0 0.13156" rpy = "0 0 1.5708"/>
-  </joint>
-  <!--
-  <joint name="joint3_to_joint2" type="revolute">
-    <axis xyz="0 0 1"/>
-    <limit effort = "1000.0" lower = "-3.14" upper = "3.14159" velocity = "0"/>
-    <parent link="joint2"/>
-    <child link="joint3"/>
-    <origin xyz= "0 0  0" rpy = "0 1.5708 -1.5708"/>
-  </joint>
-  <joint name="joint4_to_joint3" type="revolute">
-    <axis xyz=" 0 0 1"/>
-    <limit effort = "1000.0" lower = "-3.14" upper = "3.14159" velocity = "0"/>
-    <parent link="joint3"/>
-    <child link="joint4"/>
-    <origin xyz= "  -0.1104 0 0   " rpy = "0 0 0"/>
-  </joint>
-  <joint name="joint5_to_joint4" type="revolute">
-    <axis xyz=" 0 0 1"/>
-    <limit effort = "1000.0" lower = "-3.14" upper = "3.14159" velocity = "0"/>
-    <parent link="joint4"/>
-    <child link="joint5"/>
-    <origin xyz= "-0.096 0 0.06462" rpy = "0 0 -1.5708"/>
-  </joint>
-  <joint name="joint6_to_joint5" type="revolute">
-    <axis xyz="0 0 1"/>
-    <limit effort = "1000.0" lower = "-3.14" upper = "3.14159" velocity = "0"/>
-    <parent link="joint5"/>
-    <child link="joint6"/>
-    <origin xyz= "0 -0.07318 0" rpy = "1.5708 -1.5708 0"/>
-  </joint>
-  <joint name="joint6output_to_joint6" type="revolute">
-    <axis xyz="0 0 1"/>
-    <limit effort = "1000.0" lower = "-3.14" upper = "3.14159" velocity = "0"/>
-    <parent link="joint6"/>
-    <child link="joint6_flange"/>
-    <origin xyz= "0 0.0456 0" rpy = "-1.5708 0 0"/>
-  </joint>
-  -->
-  <transmission name="left_track_trans" type="SimpleTransmission">
-    <type>transmission_interface/SimpleTransmission</type>
-    <joint name="left_track_motor">
-      <hardwareInterface>hardware_interface/EffortJointInterface</hardwareInterface>
-    </joint>
-    <actuator name="left_track_motor_drive">
-      <mechanicalReduction>1</mechanicalReduction>
-    </actuator>
-  </transmission>
-  <transmission name="right_track_trans" type="SimpleTransmission">
-    <type>transmission_interface/SimpleTransmission</type>
-    <joint name="right_track_motor">
-      <hardwareInterface>hardware_interface/EffortJointInterface</hardwareInterface>
-    </joint>
-    <actuator name="right_track_motor_drive">
-      <mechanicalReduction>1</mechanicalReduction>
-    </actuator>
-  </transmission>
   <gazebo>
     <plugin name="gazebo_ros_control" filename="libgazebo_ros_control.so">
-      <robotNamespace></robotNamespace>
-    </plugin>
-    <plugin filename="libSimpleTrackedVehiclePlugin.so" name="simple_tracked_vehicle">
-      <body>base_link</body>
-      <left_track>left_track</left_track>
-      <right_track>right_track</right_track>
-      <track_mu>0.65</track_mu>
-      <track_mu2>0.85</track_mu2>
-      <tracks_separation>0.19</tracks_separation>
-      <robot_namespace>chimera</robot_namespace>
-    </plugin>
-    <plugin name='tracked_vehicle_interface' filename='libgazebo_ros_tracked_vehicle_interface.so'>
-      <commandROSTopic>/chimera/cmd_vel</commandROSTopic>
-      <commandIGNTopic>~/chimera/cmd_vel_twist</commandIGNTopic>
-      <robotBaseFrame>base_link</robotBaseFrame>
-      <tracks_separation>0.19</tracks_separation>
-      <publishOdomTF>false</publishOdomTF>
+      <robotNamespace>/chimera</robotNamespace>
     </plugin>
   </gazebo>
