Commit message: Configuration and controllers for working simulation in Gazebo.

File: chimera_description/urdf/chimera.urdf.xacro (robot description, xacro)
@@ -33,5 +33,5 @@
   <gazebo>
     <plugin name="gazebo_ros_control" filename="libgazebo_ros_control.so">
-      <robotNamespace>/chimera</robotNamespace>
+      <robotNamespace>/</robotNamespace>
     </plugin>
   </gazebo>

File: chimera_description/urdf/gripper.urdf.xacro (robot description, xacro)
@@ -2,5 +2,5 @@
 <robot xmlns:xacro="http://www.ros.org/wiki/xacro">
   <xacro:include filename="$(find chimera_description)/urdf/inertial.xacro"/>
-  <xacro:macro name="gripper" params="end_effector_link originxyz originrpy">
+  <xacro:macro name="gripper" params="wrist_link originxyz originrpy">
     <link name="gripper_base">
       <visual>
@@ -19,5 +19,5 @@
 	<origin xyz = "0.0 0 0 " rpy = " 0 0 0"/>
       </collision>
-      <xacro:box_inertial m="0.1" w="0.01" d="0.01" h="0.01"/>
+      <xacro:box_inertial m="0.025" w="0.1" d="0.1" h="0.1"/>
     </link>
     <link name="left_finger">
@@ -37,5 +37,5 @@
 	<origin xyz = "0.0 0 0 " rpy = " 0 0 0"/>
       </collision>
-      <xacro:box_inertial m="0.05" w="0.005" d="0.005" h="0.005"/>
+      <xacro:box_inertial m="0.01" w="0.1" d="0.1" h="0.1"/>
     </link>
     <link name="right_finger">
@@ -47,5 +47,5 @@
 	<material name="">
 	  <color rgba="0.7 0.7 0.7 1"/>
-      </material>
+	</material>
       </visual>
       <collision>
@@ -55,8 +55,8 @@
 	<origin xyz = "0.0 0 0 " rpy = " 0 0 0"/>
       </collision>
-      <xacro:box_inertial m="0.05" w="0.005" d="0.005" h="0.005"/>
+      <xacro:box_inertial m="0.01" w="0.1" d="0.1" h="0.1"/>
     </link>
     <joint name="gripper_base_joint" type="fixed">
-      <parent link="${end_effector_link}"/>
+      <parent link="${wrist_link}"/>
       <child link="gripper_base"/>
       <origin xyz="${originxyz}" rpy="${originrpy}"/>
@@ -64,16 +64,34 @@
     <joint name="right_finger_joint" type="revolute">
       <axis xyz="0 0 -1"/>
-      <limit effort = "10.0" lower = "0.0" upper = "0.75" velocity = "0"/>
+      <limit effort = "1.0" lower = "0.0" upper = "0.75" velocity = "1.0"/>
       <parent link="gripper_base"/>
       <child link="right_finger"/>
-      <origin xyz= "0 -0.008 0.00602" rpy = "0 0 0"/>
+      <origin xyz= "0.0 -0.008 0.00602" rpy = "0 0 0"/>
     </joint>
     <joint name="left_finger_joint" type="revolute">
+      <mimic joint="right_finger_joint"/>
       <axis xyz="0 0 1"/>
-      <limit effort = "10.0" lower = "0.0" upper = "0.75" velocity = "0"/>
+      <limit effort = "1.0" lower = "0.0" upper = "0.75" velocity = "1.0"/>
       <parent link="gripper_base"/>
       <child link="left_finger"/>
-      <origin xyz= "0 -0.008 0.00602" rpy = "0 0 0"/>
+      <origin xyz= "0.0 -0.008 0.00602" rpy = "0 0 0"/>
     </joint>
+    <!-- TODO: Might still need both transmissions? -->
+    <transmission name="trans_hand">
+      <type>transmission_interface/SimpleTransmission</type>
+      <joint name="right_finger_joint">
+        <hardwareInterface>hardware_interface/EffortJointInterface</hardwareInterface>
+      </joint>
+      <actuator name="hand_motor">
+        <hardwareInterface>hardware_interface/EffortJointInterface</hardwareInterface>
+        <mechanicalReduction>1</mechanicalReduction>
+      </actuator>
+    </transmission>
+    <gazebo>
+      <plugin name="mimic_joints" filename="libroboticsgroup_upatras_gazebo_mimic_joint_plugin.so">
+	<joint>right_finger_joint</joint>
+	<mimicJoint>left_finger_joint</mimicJoint>
+      </plugin>
+    </gazebo>
   </xacro:macro>
 </robot>

File: chimera_description/urdf/mycobot280_arduino.urdf.xacro (robot description, xacro)
@@ -17,5 +17,5 @@
         <origin xyz = "0.0 0 0 " rpy = " 0 0 3.14159"/>
       </collision>
-      <xacro:box_inertial m="0.25" w="0.1" d="0.1" h="0.1"/>
+      <xacro:hcylinder_inertial m="0.75" r="0.05" h="0.07"/>
     </link>
     <link name="link2">
@@ -32,5 +32,5 @@
 	<origin xyz = "0.0 0 -0.06096 " rpy = " 0 0 -1.5708"/>
       </collision>
-      <xacro:hcylinder_inertial m="0.1" r="0.025" h="0.087"/>
+      <xacro:hcylinder_inertial m="0.2" r="0.05" h="0.08"/>
     </link>
     <link name="link3">
@@ -47,5 +47,5 @@
 	<origin xyz = "0.0 0 0.03256 " rpy = " 0 -1.5708 0"/>
       </collision>
-      <xacro:hcylinder_inertial m="0.2" r="0.03" h="0.155"/>
+      <xacro:hcylinder_inertial m="0.4" r="0.05" h="0.155"/>
     </link>
     <link name="link4">
@@ -62,5 +62,5 @@
 	<origin xyz = "0.0 0 0.03056 " rpy = " 0 -1.5708 0"/>
       </collision>
-      <xacro:hcylinder_inertial m="0.18" r="0.0275" h="0.136"/>
+      <xacro:hcylinder_inertial m="0.4" r="0.05" h="0.155"/>
     </link>
     <link name="link5">
@@ -77,5 +77,5 @@
 	<origin xyz = "0.0 0 -0.03356 " rpy = " -1.5708 0 0"/>
       </collision>
-      <xacro:hcylinder_inertial m="0.1" r="0.0275" h="0.06"/>
+      <xacro:hcylinder_inertial m="0.2" r="0.05" h="0.05"/>
     </link>
     <link name="link6">
@@ -92,10 +92,10 @@
 	<origin xyz = "0 0.00 -0.038 " rpy = " 0 0 0"/>
       </collision>
-      <xacro:hcylinder_inertial m="0.1" r="0.018" h="0.06"/>
-    </link>
-    <link name="end_effector_link">
-      <visual>
-	<geometry>
-	  <mesh filename="package://chimera_description/meshes/end_effector.dae"/>
+      <xacro:hcylinder_inertial m="0.5" r="0.05" h="0.06"/>
+    </link>
+    <link name="wrist_link">
+      <visual>
+	<geometry>
+	  <mesh filename="package://chimera_description/meshes/wrist.dae"/>
 	</geometry>
 	<origin xyz = "0.0 0 -0.012 " rpy = " 0 0 0"/>
@@ -103,12 +103,12 @@
       <collision>
 	<geometry>
-	  <mesh filename="package://chimera_description/meshes/end_effector.dae"/>
+	  <mesh filename="package://chimera_description/meshes/wrist.dae"/>
 	</geometry>
 	<origin xyz = "0.0 0 -0.012 " rpy = " 0 0 0"/>
       </collision>
-      <xacro:hcylinder_inertial m="0.05" r="0.018" h="0.02"/>
-    </link>
-    <xacro:gripper end_effector_link="end_effector_link"
-			originxyz="0.0 0.012 0.027" originrpy="1.570796 3.14159 0"/>
+      <xacro:hcylinder_inertial m="0.1" r="0.02" h="0.005"/>
+    </link>
+    <xacro:gripper wrist_link="wrist_link"
+		   originxyz="0.0 0.012 0.027" originrpy="1.570796 3.14159 0"/>
     <joint name="arm_to_baselink" type="fixed">
       <parent link="${moving_base_link}"/>
@@ -118,44 +118,110 @@
     <joint name="joint21" type="revolute">
       <axis xyz="0 0 1"/>
-      <limit effort = "1000.0" lower = "-3.14" upper = "3.14159" velocity = "0"/>
+      <limit effort = "1000.0" lower = "-3.14" upper = "3.14159" velocity = "0.1"/>
       <parent link="link1"/>
       <child link="link2"/>
       <origin xyz= "0 0 0.13156" rpy = "0 0 1.5708"/>
+      <dynamics damping="1.0e-6" friction="2.0e-1" />
     </joint>
     <joint name="joint32" type="revolute">
       <axis xyz="0 0 1"/>
-      <limit effort = "1000.0" lower = "-3.14" upper = "3.14159" velocity = "0"/>
+      <limit effort = "1000.0" lower = "-3.14" upper = "3.14159" velocity = "0.25"/>
       <parent link="link2"/>
       <child link="link3"/>
       <origin xyz= "0 0  0" rpy = "0 1.5708 -1.5708"/>
+      <dynamics damping="1.0e-6" friction="2.0e-1" />
     </joint>
     <joint name="joint43" type="revolute">
       <axis xyz=" 0 0 1"/>
-      <limit effort = "1000.0" lower = "-3.14" upper = "3.14159" velocity = "0"/>
+      <limit effort = "1000.0" lower = "-3.14" upper = "3.14159" velocity = "0.25"/>
       <parent link="link3"/>
       <child link="link4"/>
       <origin xyz= "  -0.1104 0 0   " rpy = "0 0 0"/>
+      <dynamics damping="1.0e-6" friction="2.0e-1" />
     </joint>
     <joint name="joint54" type="revolute">
       <axis xyz=" 0 0 1"/>
-      <limit effort = "1000.0" lower = "-3.14" upper = "3.14159" velocity = "0"/>
+      <limit effort = "1000.0" lower = "-3.14" upper = "3.14159" velocity = "0.25"/>
       <parent link="link4"/>
       <child link="link5"/>
       <origin xyz= "-0.096 0 0.06462" rpy = "0 0 -1.5708"/>
+      <dynamics damping="1.0e-6" friction="2.0e-1" />
     </joint>
     <joint name="joint65" type="revolute">
       <axis xyz="0 0 1"/>
-      <limit effort = "1000.0" lower = "-3.14" upper = "3.14159" velocity = "0"/>
+      <limit effort = "1000.0" lower = "-3.14" upper = "3.14159" velocity = "0.25"/>
       <parent link="link5"/>
       <child link="link6"/>
       <origin xyz= "0 -0.07318 0" rpy = "1.5708 -1.5708 0"/>
-    </joint>
-    <joint name="end_effector_joint" type="revolute">
-      <axis xyz="0 0 1"/>
-      <limit effort = "1000.0" lower = "-3.14" upper = "3.14159" velocity = "0"/>
+      <dynamics damping="1.0e-6" friction="2.0e-1" />
+    </joint>
+    <joint name="wrist_joint" type="revolute">
+      <axis xyz="0 0 1"/>
+      <limit effort = "1000.0" lower = "-3.14" upper = "3.14159" velocity = "0.25"/>
       <parent link="link6"/>
-      <child link="end_effector_link"/>
+      <child link="wrist_link"/>
       <origin xyz= "0 0.0456 0" rpy = "-1.5708 0 0"/>
-    </joint>
+      <dynamics damping="1.0e-6" friction="2.0e-1" />
+    </joint>
+    <transmission name="trans_joint21">
+      <type>transmission_interface/SimpleTransmission</type>
+      <joint name="joint21">
+        <hardwareInterface>hardware_interface/EffortJointInterface</hardwareInterface>
+      </joint>
+      <actuator name="joint21_motor">
+        <hardwareInterface>hardware_interface/EffortJointInterface</hardwareInterface>
+        <mechanicalReduction>1</mechanicalReduction>
+      </actuator>
+    </transmission>
+    <transmission name="trans_joint32">
+      <type>transmission_interface/SimpleTransmission</type>
+      <joint name="joint32">
+        <hardwareInterface>hardware_interface/EffortJointInterface</hardwareInterface>
+      </joint>
+      <actuator name="joint32_motor">
+        <hardwareInterface>hardware_interface/EffortJointInterface</hardwareInterface>
+        <mechanicalReduction>1</mechanicalReduction>
+      </actuator>
+    </transmission>
+    <transmission name="trans_joint43">
+      <type>transmission_interface/SimpleTransmission</type>
+      <joint name="joint43">
+        <hardwareInterface>hardware_interface/EffortJointInterface</hardwareInterface>
+      </joint>
+      <actuator name="joint43_motor">
+        <hardwareInterface>hardware_interface/EffortJointInterface</hardwareInterface>
+        <mechanicalReduction>1</mechanicalReduction>
+      </actuator>
+    </transmission>
+    <transmission name="trans_joint54">
+      <type>transmission_interface/SimpleTransmission</type>
+      <joint name="joint54">
+        <hardwareInterface>hardware_interface/EffortJointInterface</hardwareInterface>
+      </joint>
+      <actuator name="joint54_motor">
+        <hardwareInterface>hardware_interface/EffortJointInterface</hardwareInterface>
+        <mechanicalReduction>1</mechanicalReduction>
+      </actuator>
+    </transmission>
+    <transmission name="trans_joint65">
+      <type>transmission_interface/SimpleTransmission</type>
+      <joint name="joint65">
+        <hardwareInterface>hardware_interface/EffortJointInterface</hardwareInterface>
+      </joint>
+      <actuator name="joint65_motor">
+        <hardwareInterface>hardware_interface/EffortJointInterface</hardwareInterface>
+        <mechanicalReduction>1</mechanicalReduction>
+      </actuator>
+    </transmission>
+    <transmission name="trans_wrist_joint">
+      <type>transmission_interface/SimpleTransmission</type>
+      <joint name="wrist_joint">
+        <hardwareInterface>hardware_interface/EffortJointInterface</hardwareInterface>
+      </joint>
+      <actuator name="wrist_joint_motor">
+        <hardwareInterface>hardware_interface/EffortJointInterface</hardwareInterface>
+        <mechanicalReduction>1</mechanicalReduction>
+      </actuator>
+    </transmission>
   </xacro:macro>
 </robot>

File: chimera_description/urdf/tracks.urdf.xacro (robot description, xacro)
@@ -100,5 +100,5 @@
     </transmission>
     <gazebo>
-      <plugin filename="libSimpleTrackedVehiclePlugin.so" name="simple_tracked_vehicle">
+      <plugin name="simple_tracked_vehicle" filename="libSimpleTrackedVehiclePlugin.so">
 	<body>base_link</body>
 	<left_track>left_track</left_track>
@@ -109,5 +109,5 @@
 	<robot_namespace>chimera</robot_namespace>
       </plugin>
-      <plugin name='tracked_vehicle_interface' filename='libgazebo_ros_tracked_vehicle_interface.so'>
+      <plugin name="tracked_vehicle_interface" filename="libgazebo_ros_tracked_vehicle_interface.so">
 	<commandROSTopic>/chimera/cmd_vel</commandROSTopic>
 	<commandIGNTopic>~/chimera/cmd_vel_twist</commandIGNTopic>

Commit message: Inital configuration for moveit and simulation. Requires some tweaks

File: chimera_description/urdf/chimera.urdf.xacro (robot description, xacro)
@@ -27,11 +27,11 @@
   <xacro:tracks />
   <joint name="base_joint" type="fixed">
-    <parent link="base_link"/>
-    <child link="base_footprint"/>
-    <origin xyz="0.0 0.0 -0.0678" rpy="0 0 0"/>
+    <parent link="base_footprint"/>
+    <child link="base_link"/>
+    <origin xyz="0.0 0.0 0.0" rpy="0 0 0"/>
   </joint>
   <gazebo>
     <plugin name="gazebo_ros_control" filename="libgazebo_ros_control.so">
-      <robotNamespace>/</robotNamespace>
+      <!--<robotNamespace>/</robotNamespace>-->
     </plugin>
   </gazebo>

File: chimera_description/urdf/tracks.urdf.xacro (robot description, xacro)
@@ -101,5 +101,5 @@
     <gazebo>
       <plugin name="simple_tracked_vehicle" filename="libSimpleTrackedVehiclePlugin.so">
-	<body>base_link</body>
+	<body>base_footprint</body>
 	<left_track>left_track</left_track>
 	<right_track>right_track</right_track>
