Commit message: hardware controller added

File: chimera_description/urdf/gripper.urdf.xacro (robot description, xacro)
@@ -64,5 +64,5 @@
     <joint name="right_finger_joint" type="revolute">
       <axis xyz="0 0 -1"/>
-      <limit effort = "1.0" lower = "0.0" upper = "0.75" velocity = "1.0"/>
+      <limit effort = "1.0" lower = "0" upper = "1.0" velocity = "1.5"/>
       <parent link="gripper_base"/>
       <child link="right_finger"/>
@@ -72,5 +72,5 @@
       <mimic joint="right_finger_joint"/>
       <axis xyz="0 0 1"/>
-      <limit effort = "1.0" lower = "0.0" upper = "0.75" velocity = "1.0"/>
+      <limit effort = "1.0" lower = "0" upper = "1.0" velocity = "1.5"/>
       <parent link="gripper_base"/>
       <child link="left_finger"/>

File: chimera_description/urdf/mycobot280_arduino.urdf.xacro (robot description, xacro)
@@ -94,4 +94,23 @@
       <xacro:hcylinder_inertial m="0.5" r="0.05" h="0.06"/>
     </link>
+     <link name="camera_link">
+      <visual>
+        <geometry>
+          <box size="0.03 0.02 0.03"/> <!-- Dimensions of the camera box -->
+        </geometry>
+        <origin xyz="0 0 0.0" rpy="0 0 1.54"/> <!-- Position and orientation of the camera -->
+      </visual>
+      <collision>
+        <geometry>
+          <box size="0.03 0.02 0.03"/> <!-- Dimensions of the camera box -->
+        </geometry>
+        <origin xyz="0 0 0" rpy="0 0 1.54"/> <!-- Position and orientation of the camera -->
+      </collision>
+    </link>
+    <joint name="wrist_to_camera_joint" type="fixed">
+      <parent link="link6"/>
+      <child link="camera_link"/>
+      <origin xyz="0 0.025 0.04" rpy="0 0 1.54"/> <!-- Position and orientation of the camera relative to the wrist -->
+    </joint>
     <link name="wrist_link">
       <visual>
@@ -118,5 +137,5 @@
     <joint name="joint21" type="revolute">
       <axis xyz="0 0 1"/>
-      <limit effort = "1000.0" lower = "-3.14" upper = "3.14159" velocity = "0.1"/>
+      <limit effort = "1000.0" lower = "-2.8" upper = "2.8" velocity = "0.1"/>
       <parent link="link1"/>
       <child link="link2"/>
@@ -126,5 +145,5 @@
     <joint name="joint32" type="revolute">
       <axis xyz="0 0 1"/>
-      <limit effort = "1000.0" lower = "-3.14" upper = "3.14159" velocity = "0.25"/>
+      <limit effort = "1000.0" lower = "-2.8" upper = "2.8" velocity = "0.25"/>
       <parent link="link2"/>
       <child link="link3"/>
@@ -134,5 +153,5 @@
     <joint name="joint43" type="revolute">
       <axis xyz=" 0 0 1"/>
-      <limit effort = "1000.0" lower = "-3.14" upper = "3.14159" velocity = "0.25"/>
+      <limit effort = "1000.0" lower = "-2.8" upper = "2.8" velocity = "0.25"/>
       <parent link="link3"/>
       <child link="link4"/>
@@ -142,5 +161,5 @@
     <joint name="joint54" type="revolute">
       <axis xyz=" 0 0 1"/>
-      <limit effort = "1000.0" lower = "-3.14" upper = "3.14159" velocity = "0.25"/>
+      <limit effort = "1000.0" lower = "-2.8" upper = "2.8" velocity = "0.25"/>
       <parent link="link4"/>
       <child link="link5"/>
@@ -150,5 +169,5 @@
     <joint name="joint65" type="revolute">
       <axis xyz="0 0 1"/>
-      <limit effort = "1000.0" lower = "-3.14" upper = "3.14159" velocity = "0.25"/>
+      <limit effort = "1000.0" lower = "-2.8" upper = "2.8" velocity = "0.25"/>
       <parent link="link5"/>
       <child link="link6"/>
@@ -158,5 +177,5 @@
     <joint name="wrist_joint" type="revolute">
       <axis xyz="0 0 1"/>
-      <limit effort = "1000.0" lower = "-3.14" upper = "3.14159" velocity = "0.25"/>
+      <limit effort = "1000.0" lower = "-3.05" upper = "3.05" velocity = "0.25"/>
       <parent link="link6"/>
       <child link="wrist_link"/>
