Commit message: Renaming joints to something that makes senes

File: chimera_description/urdf/mycobot280_arduino.urdf.xacro (robot description, xacro)
@@ -3,8 +3,8 @@
   <xacro:include filename="$(find chimera_description)/urdf/inertial.xacro"/>
   <xacro:macro name="my_cobot_arm" params="moving_base_link originxyz originrpy">
-    <link name="joint1">
+    <link name="link1">
       <visual>
 	<geometry>
-	  <mesh filename="package://chimera_description/meshes/joint1.dae"/>
+	  <mesh filename="package://chimera_description/meshes/link1.dae"/>
 	</geometry>
 	<origin xyz = "0.0 0 0 " rpy = " 0 0 3.14159"/>
@@ -12,5 +12,5 @@
       <collision>
 	<geometry>
-	  <mesh filename="package://chimera_description/meshes/joint1.dae"/>
+	  <mesh filename="package://chimera_description/meshes/link1.dae"/>
         </geometry>
         <origin xyz = "0.0 0 0 " rpy = " 0 0 3.14159"/>
@@ -18,8 +18,8 @@
       <xacro:box_inertial m="0.25" w="0.1" d="0.1" h="0.1"/>
     </link>
-    <link name="joint2">
+    <link name="link2">
       <visual>
 	<geometry>
-	  <mesh filename="package://chimera_description/meshes/joint2.dae"/>
+	  <mesh filename="package://chimera_description/meshes/link2.dae"/>
 	</geometry>
 	<origin xyz = "0.0 0 -0.06096 " rpy = " 0 0 -1.5708"/>
@@ -27,5 +27,5 @@
       <collision>
 	<geometry>
-	  <mesh filename="package://chimera_description/meshes/joint2.dae"/>
+	  <mesh filename="package://chimera_description/meshes/link2.dae"/>
 	</geometry>
 	<origin xyz = "0.0 0 -0.06096 " rpy = " 0 0 -1.5708"/>
@@ -33,8 +33,8 @@
       <xacro:hcylinder_inertial m="0.1" r="0.025" h="0.087"/>
     </link>
-    <link name="joint3">
+    <link name="link3">
       <visual>
 	<geometry>
-	  <mesh filename="package://chimera_description/meshes/joint3.dae"/>
+	  <mesh filename="package://chimera_description/meshes/link3.dae"/>
 	</geometry>
 	<origin xyz = "0.0 0 0.03256 " rpy = " 0 -1.5708 0"/>
@@ -42,5 +42,5 @@
       <collision>
 	<geometry>
-	  <mesh filename="package://chimera_description/meshes/joint3.dae"/>
+	  <mesh filename="package://chimera_description/meshes/link3.dae"/>
 	</geometry>
 	<origin xyz = "0.0 0 0.03256 " rpy = " 0 -1.5708 0"/>
@@ -48,8 +48,8 @@
       <xacro:hcylinder_inertial m="0.2" r="0.03" h="0.155"/>
     </link>
-    <link name="joint4">
+    <link name="link4">
       <visual>
 	<geometry>
-	  <mesh filename="package://chimera_description/meshes/joint4.dae"/>
+	  <mesh filename="package://chimera_description/meshes/link4.dae"/>
 	</geometry>
 	<origin xyz = "0.0 0 0.03056 " rpy = " 0 -1.5708 0"/>
@@ -57,5 +57,5 @@
       <collision>
 	<geometry>
-	  <mesh filename="package://chimera_description/meshes/joint4.dae"/>
+	  <mesh filename="package://chimera_description/meshes/link4.dae"/>
 	</geometry>
 	<origin xyz = "0.0 0 0.03056 " rpy = " 0 -1.5708 0"/>
@@ -63,8 +63,8 @@
       <xacro:hcylinder_inertial m="0.18" r="0.0275" h="0.136"/>
     </link>
-    <link name="joint5">
+    <link name="link5">
       <visual>
 	<geometry>
-	  <mesh filename="package://chimera_description/meshes/joint5.dae"/>
+	  <mesh filename="package://chimera_description/meshes/link5.dae"/>
 	</geometry>
 	<origin xyz = "0.0 0 -0.03356 " rpy = " -1.5708 0 0"/>
@@ -72,5 +72,5 @@
       <collision>
 	<geometry>
-	  <mesh filename="package://chimera_description/meshes/joint5.dae"/>
+	  <mesh filename="package://chimera_description/meshes/link5.dae"/>
 	</geometry>
 	<origin xyz = "0.0 0 -0.03356 " rpy = " -1.5708 0 0"/>
@@ -78,8 +78,8 @@
       <xacro:hcylinder_inertial m="0.1" r="0.0275" h="0.06"/>
     </link>
-    <link name="joint6">
+    <link name="link6">
       <visual>
 	<geometry>
-	  <mesh filename="package://chimera_description/meshes/joint6.dae"/>
+	  <mesh filename="package://chimera_description/meshes/link6.dae"/>
 	</geometry>
 	<origin xyz = "0 0.00 -0.038 " rpy = " 0 0 0"/>
@@ -87,5 +87,5 @@
       <collision>
 	<geometry>
-	  <mesh filename="package://chimera_description/meshes/joint6.dae"/>
+	  <mesh filename="package://chimera_description/meshes/link6.dae"/>
 	</geometry>
 	<origin xyz = "0 0.00 -0.038 " rpy = " 0 0 0"/>
@@ -93,8 +93,8 @@
       <xacro:hcylinder_inertial m="0.1" r="0.018" h="0.06"/>
     </link>
-    <link name="joint6_flange">
+    <link name="end_effector_link">
       <visual>
 	<geometry>
-	  <mesh filename="package://chimera_description/meshes/joint7.dae"/>
+	  <mesh filename="package://chimera_description/meshes/end_effector.dae"/>
 	</geometry>
 	<origin xyz = "0.0 0 -0.012 " rpy = " 0 0 0"/>
@@ -102,5 +102,5 @@
       <collision>
 	<geometry>
-	  <mesh filename="package://chimera_description/meshes/joint7.dae"/>
+	  <mesh filename="package://chimera_description/meshes/end_effector.dae"/>
 	</geometry>
 	<origin xyz = "0.0 0 -0.012 " rpy = " 0 0 0"/>
@@ -110,47 +110,47 @@
     <joint name="arm_to_baselink" type="fixed">
       <parent link="${moving_base_link}"/>
-      <child link="joint1"/>
+      <child link="link1"/>
       <origin xyz="${originxyz}" rpy="${originrpy}"/>
     </joint>
-    <joint name="joint2_to_joint1" type="revolute">
+    <joint name="joint21" type="revolute">
       <axis xyz="0 0 1"/>
       <limit effort = "1000.0" lower = "-3.14" upper = "3.14159" velocity = "0"/>
-      <parent link="joint1"/>
-      <child link="joint2"/>
+      <parent link="link1"/>
+      <child link="link2"/>
       <origin xyz= "0 0 0.13156" rpy = "0 0 1.5708"/>
     </joint>
-    <joint name="joint3_to_joint2" type="revolute">
+    <joint name="joint32" type="revolute">
       <axis xyz="0 0 1"/>
       <limit effort = "1000.0" lower = "-3.14" upper = "3.14159" velocity = "0"/>
-      <parent link="joint2"/>
-      <child link="joint3"/>
+      <parent link="link2"/>
+      <child link="link3"/>
       <origin xyz= "0 0  0" rpy = "0 1.5708 -1.5708"/>
     </joint>
-    <joint name="joint4_to_joint3" type="revolute">
+    <joint name="joint43" type="revolute">
       <axis xyz=" 0 0 1"/>
       <limit effort = "1000.0" lower = "-3.14" upper = "3.14159" velocity = "0"/>
-      <parent link="joint3"/>
-      <child link="joint4"/>
+      <parent link="link3"/>
+      <child link="link4"/>
       <origin xyz= "  -0.1104 0 0   " rpy = "0 0 0"/>
     </joint>
-    <joint name="joint5_to_joint4" type="revolute">
+    <joint name="joint54" type="revolute">
       <axis xyz=" 0 0 1"/>
       <limit effort = "1000.0" lower = "-3.14" upper = "3.14159" velocity = "0"/>
-      <parent link="joint4"/>
-      <child link="joint5"/>
+      <parent link="link4"/>
+      <child link="link5"/>
       <origin xyz= "-0.096 0 0.06462" rpy = "0 0 -1.5708"/>
     </joint>
-    <joint name="joint6_to_joint5" type="revolute">
+    <joint name="joint65" type="revolute">
       <axis xyz="0 0 1"/>
       <limit effort = "1000.0" lower = "-3.14" upper = "3.14159" velocity = "0"/>
-      <parent link="joint5"/>
-      <child link="joint6"/>
+      <parent link="link5"/>
+      <child link="link6"/>
       <origin xyz= "0 -0.07318 0" rpy = "1.5708 -1.5708 0"/>
     </joint>
-    <joint name="joint6output_to_joint6" type="revolute">
+    <joint name="end_effector_joint" type="revolute">
       <axis xyz="0 0 1"/>
       <limit effort = "1000.0" lower = "-3.14" upper = "3.14159" velocity = "0"/>
-      <parent link="joint6"/>
-      <child link="joint6_flange"/>
+      <parent link="link6"/>
+      <child link="end_effector_link"/>
       <origin xyz= "0 0.0456 0" rpy = "-1.5708 0 0"/>
     </joint>

Commit message: Update mycobot280_arduino.urdf.xacro

File: chimera_description/urdf/mycobot280_arduino.urdf.xacro (robot description, xacro)
@@ -111,5 +111,5 @@
       <parent link="link6"/>
       <child link="camera_link"/>
-      <origin xyz="0 0.025 0.04" rpy="0 0 1.54"/> <!-- Position and orientation of the camera relative to the wrist -->
+      <origin xyz="0 -0.035 0.035" rpy="0 0 1.54"/> <!-- Position and orientation of the camera relative to the wrist -->
     </joint>
     <link name="wrist_link">
